Commit message: 提交

File: 模型/仿真模型/ROS2/balance_car_description/urdf/balance_car.urdf (robot description, URDF)
Before this commit: robot balance_car_zd2808, 3 links, 2 joints
Links:
- link left_wheel: geometry collision cylinder length=.028 radius=0.0325; visual mesh filename=package://balance_car_description/meshes/right_wheel.stl scale=1 1 1
- link right_wheel: geometry collision cylinder length=.028 radius=0.0325; visual mesh filename=package://balance_car_description/meshes/left_wheel.stl scale=1 1 1
Joints:
- joint left_wheel_joint: axis 0 1 0 -> -1 0 0; origin xyz=0 0.0662682 0 rpy=0 0 0 -> xyz=-0.0662682 0 0 rpy=0 0 0
- joint right_wheel_joint: axis 0 1 0 -> -1 0 0; origin xyz=0 -0.0662682 0 rpy=0 0 0 -> xyz=0.0662682 0 0 rpy=0 0 0

File: 模型/仿真模型/通用URDF/urdf/balance_car.urdf (robot description, URDF)
Before this commit: robot balance_car_zd2808, 3 links, 2 joints
Links:
- link left_wheel: geometry collision cylinder length=.028 radius=0.0325; visual mesh filename=../meshes/right_wheel.stl scale=1 1 1
- link right_wheel: geometry collision cylinder length=.028 radius=0.0325; visual mesh filename=../meshes/left_wheel.stl scale=1 1 1
Joints:
- joint left_wheel_joint: axis 0 1 0 -> -1 0 0; origin xyz=0 0.0662682 0 rpy=0 0 0 -> xyz=-0.0662682 0 0 rpy=0 0 0
- joint right_wheel_joint: axis 0 1 0 -> -1 0 0; origin xyz=0 -0.0662682 0 rpy=0 0 0 -> xyz=0.0662682 0 0 rpy=0 0 0
